File: hardware/schematic/final year project.kicad_sch (KiCad schematic)
At the start: 0 parts

Commit message: Completed power supply schematic
Parts:
- added BT1: Battery_Cell, symbol Device:Battery_Cell
- added D1: LED, symbol Device:LED
- added R1: 1k, symbol Device:R
- added SW1: SW_SPST, symbol Switch:SW_SPST
- added TP1: VBAT, symbol Connector:TestPoint
- added TP2: 3V3, symbol Connector:TestPoint
- added U1: (no value), symbol Battery management cus:TPTP4056_USB_C_PROTECTED
- added U2: (no value), symbol Voltage Regulator:TPS63020_3V3_MODULE
Connections:
- new net: D1.2 (A), R1.2
- new net: SW1.2 (B), TP1.1, U2.1 (VIN+)
- new net: SW1.1 (A), U1.3 (OUT+)
- new net: U1.4 (OUT-), U2.2 (VIN-)
- new net: BT1.1 (+), U1.5 (B+)
- new net: BT1.2 (-), U1.6 (B-)
- new net +3.3V: R1.1, TP2.1, U2.3 (VOUT)
- new net +5V: U1.1 (IN+)
- new net GND: D1.1 (K), U1.2 (IN-), U2.4 (VOUT-)
Other:
- note added: "Power Supply"
